Commit message: Important bug fixes to have the package working as in ROSConFr 2023wq

File: odri_dual_motor_testbed_description/ros2_control/system_dual_motor_testbed.ros2_control.xacro (robot description, xacro)
@@ -20,10 +20,10 @@
             <param name="odri_config_yaml">${prop_dual_motor_testbed_config_yaml}</param>
             <param name="desired_starting_position">0.0 0.0</param>
-            <param name="default_joint_cmd">FL_HAA 0.0 0.0 0.0 3.0 0.05 FR_HAA 0.0 0.0 0.0 3.0 0.05</param>
-            <param name="default_joint_state">FL_HAA 0.0 0.0 0.0 3.0 0.05 FR_HAA 0.0 0.0 0.0 3.0 0.05</param>
+            <param name="default_joint_cmd">odri_dm_tb_kt_left_joint 0.0 0.0 0.0 3.0 0.05 odri_dm_tb_kt_right_joint 0.0 0.0 0.0 3.0 0.05</param>
+            <param name="default_joint_state">odri_dm_tb_kt_left_joint 0.0 0.0 0.0 3.0 0.05 odri_dm_tb_kt_right_joint 0.0 0.0 0.0 3.0 0.05</param>
             </xacro:unless>
         </hardware>
       </xacro:unless>
-      <joint name="FL_HAA">
+      <joint name="odri_dm_tb_kt_left_joint">
         <command_interface name="position">
           <param name="min">-0.9</param>
@@ -52,5 +52,5 @@
         <state_interface name="gain_kd"/>
       </joint>
-      <joint name="FR_HAA">
+      <joint name="odri_dm_tb_kt_right_joint">
         <command_interface name="position">
           <param name="min">-0.9</param>

File: odri_dual_motor_testbed_description/urdf/base.urdf.xacro (robot description, xacro)
@@ -14,5 +14,5 @@
 <robot xmlns:xacro="http://ros.org/wiki/xacro">
   <xacro:include filename="$(find odri_dual_motor_testbed_description)/urdf/wheel.urdf.xacro" />
-  <xacro:macro name="odri_dual_motor_testbed_kin_tree" params="name parent ">
+  <xacro:macro name="odri_dual_motor_testbed_kin_tree" params="name parent">
     <!--************************-->
     <!--   BASE    -->
