Commit message: [odri_dual_motor_testbed_description] Fix wrong value for the position of the rotor.

File: odri_dual_motor_testbed_description/urdf/fivebar_2dof.urdf.xacro (robot description, xacro)
@@ -23,4 +23,8 @@
      from the previous revision of this file, so the arms never self-collide.
   5. ros2_control + Gazebo plugin blocks appended (not part of the export).
+  6. motor_1 / motor_2 origin yaw set to 0 (exported: 0.662203 / -0.0662491),
+     so that theta = 0 matches the encoder zero (both cranks parallel, along
+     +y of `case`). This changes phi1/phi2/psi1/psi2 of the analytical model;
+     see five_bar_mgd_spec.md section 2.
   NOTE on orientation: the mechanism plane is the (x,y) plane of `case`, with
   both motor axes along -z. With the base plate flat on the ground this is a
@@ -184,5 +188,5 @@
     </collision>
   </link>
-  <!-- Link rotor (left crank: motor rotor + arm_l1) -->
+  <!-- Link rotor (left crank motor rotor + arm_l1) -->
   <link name="rotor">
     <inertial>
@@ -302,5 +306,5 @@
   <!-- Joint from case to rotor (actuated, theta1) -->
   <joint name="motor_1" type="continuous">
-    <origin xyz="-0.0421006 0.0302628 0.00805311" rpy="-3.14159 0 0.662203"/>
+    <origin xyz="-0.0421006 0.0302628 0.00805311" rpy="-3.14159 0 0.0"/>
     <parent link="case"/>
     <child link="rotor"/>
@@ -308,5 +312,5 @@
     <limit effort="10" velocity="10"/>
   </joint>
-  <!-- Link rotor_2 (right crank: motor rotor + arm_r1) -->
+  <!-- Link rotor_2 (right crank motor rotor + arm_r1) -->
   <link name="rotor_2">
     <inertial>
@@ -426,5 +430,5 @@
   <!-- Joint from case to rotor_2 (actuated, theta2) -->
   <joint name="motor_2" type="continuous">
-    <origin xyz="0.0578994 0.0302628 0.00805311" rpy="3.14159 0 -0.0662491"/>
+    <origin xyz="0.0578994 0.0302628 0.00805311" rpy="3.14159 0 -0.0"/>
     <parent link="case"/>
     <child link="rotor_2"/>
