Commit message: Add new model provided by Thomas Flayols.

File: odri_dual_motor_testbed_description/robots/odri_dual_motor_testbed.urdf.xacro (robot description, xacro)
@@ -20,5 +20,6 @@
   <xacro:include filename="$(find odri_dual_motor_testbed_description)/ros2_control/system_dual_motor_testbed.ros2_control.xacro" />
   <xacro:odri_dual_motor_testbed_ros2_control
-    use_sim="$(arg use_sim)" name="odri_dm_tb_kt"/>
+      use_sim="$(arg use_sim)" name="odri_dm_tb_kt"/>
+  <link name="world"/>
   <xacro:include filename="$(find odri_dual_motor_testbed_description)/urdf/base.urdf.xacro" />
   <xacro:odri_dual_motor_testbed_kin_tree

File: odri_dual_motor_testbed_description/urdf/base.urdf.xacro (robot description, xacro)
@@ -42,4 +42,9 @@
       </collision>
     </link>
+    <joint name="${name}_in_${parent}" type="fixed">
+      <parent link="${parent}" />
+      <child link="base_footprint" />
+      <origin xyz="0.0 0.0 0.01" rpy ="0.0 0.0 0.0"/>
+    </joint>
     <joint name="${name}_1_joint" type="fixed">
       <parent link="base_footprint" />
