Commit message: [

File: odri_dual_motor_testbed_description/robots/fivebar_2dof_robot_gazebo.urdf.xacro (robot description, xacro)
@@ -26,3 +26,75 @@
     <origin xyz="0.0 0.0 0.001" rpy ="0.0 0.0 0.0"/>
   </joint>
+    <ros2_control name="GazeboOdriSimSystem" type="system">
+    <hardware>
+      <plugin>odri_gz_ros2_control/GazeboOdriSimSystem</plugin>
+    </hardware>
+    <joint name="motorL">
+      <command_interface name="position" />
+      <command_interface name="velocity" />
+      <command_interface name="effort" />
+      <command_interface name="gain_kp" />
+      <command_interface name="gain_kd" />
+      <state_interface name="velocity" />
+      <state_interface name="position" />
+      <state_interface name="effort" />
+    </joint>
+    <joint name="motorR">
+      <command_interface name="position" />
+      <command_interface name="velocity" />
+      <command_interface name="effort" />
+      <command_interface name="gain_kp" />
+      <command_interface name="gain_kd" />
+      <state_interface name="velocity" />
+      <state_interface name="position" />
+      <state_interface name="effort" />
+    </joint>
+    <joint name="elbowL">
+      <state_interface name="velocity" />
+      <state_interface name="position" />
+      <state_interface name="effort" />
+    </joint>
+    <joint name="elbowR">
+      <state_interface name="velocity" />
+      <state_interface name="position" />
+      <state_interface name="effort" />
+    </joint>
+  </ros2_control>
+  <gazebo>
+    <plugin filename="odri_gz_ros2_control-system" name="odri_gz_ros2_control::GazeboOdriSimROS2ControlPlugin">
+      <parameters>$(arg controller_params_file)</parameters>
+      <ros>
+        <namespace>$(arg robot_namespace)</namespace>
+      </ros>
+    </plugin>
+  </gazebo>
+  <!-- ================================================================ -->
+  <!--      Gazebo Harmonic (gz-sim8) system plugin for five-bar loop closure. -->
+  <!--      Exact direct geometric model: reads motorL/motorR and imposes -->
+  <!--      elbowL/elbowR via Joint::ResetPosition every step. -->
+  <!--      See five_bar_mgd_spec.md at the repository root. -->
+  <!--      ================================================================ -->
+  <gazebo>
+    <plugin filename="libFiveBarClosurePlugin.so"
+            name="odri_gz::FiveBarClosurePlugin">
+      <!-- Actuated joints (inputs, theta1/theta2). -->
+      <motor_joint1>motorL</motor_joint1>
+      <motor_joint2>motorR</motor_joint2>
+      <!-- Passive joints (outputs, beta1/beta2), imposed exactly. -->
+      <elbow_joint1>elbowL</elbow_joint1>
+      <elbow_joint2>elbowR</elbow_joint2>
+      <!-- Geometry parameters (verified numerically, see
+           five_bar_mgd_spec.md section 2). -->
+      <a_x>-0.065</a_x>
+      <a_z>0</a_z>
+      <b_x>0.065</b_x>
+      <b_z>0</b_z>
+      <l1>0.06</l1>
+      <l2>0.125</l2>
+      <phi1>3.14159265358979323846</phi1>
+      <phi2>1.9504681943696776</phi2>
+      <psi1>1.1061036468685321</psi1>
+      <psi2>2.6769066384729094</psi2>
+    </plugin>
+  </gazebo>
 </robot>

File: odri_dual_motor_testbed_description/urdf/dual_flywheel.urdf.xacro (robot description, xacro)
@@ -13,5 +13,5 @@
      same as for the five-bar model (see fivebar_2dof.urdf.xacro).
   3. The ros2_control block + odri_gz_ros2_control plugin live in
-     ros2_control/system_dual_flywheel.ros2_control.xacro, included
+     ros2_control/system_pico_dual_drv8316c.ros2_control.xacro, included
      separately by robots/dual_flywheel_robot.urdf.xacro.
   This mechanism has no closed kinematic loop: motor_1/motor_2 directly
