Commit message: [odri_dual_motor_testbed_description] Improved organization of the xacro and urdf files + cleaning.

File: odri_dual_motor_testbed_description/robots/dual_flywheel_robot.urdf.xacro (robot description, xacro)
@@ -9,4 +9,5 @@
        single-robot behaviour is unchanged. -->
   <xacro:arg name="robot_namespace" default=""/>
+  <xacro:arg name="gz_sim" default="false"/>
   <link name="world"/>
   <xacro:include filename="$(find odri_dual_motor_testbed_description)/urdf/dual_flywheel.urdf.xacro" />
@@ -16,7 +17,13 @@
     <origin xyz="0.0 0.0 0.001" rpy ="0.0 0.0 0.0"/>
   </joint>
-  <xacro:include filename="$(find odri_dual_motor_testbed_description)/ros2_control/system_pico_dual_drv8316c.ros2_control.xacro" />
-  <xacro:pico_dual_drv8316c_ros2_control
-      name="picodualdrv8316c"
-      />
+  <xacro:if value="$(arg gz_sim)">
+    <xacro:include filename="$(find odri_dual_motor_testbed_description)/gazebo/gazebo_dual_flywheel.urdf.xacro" />
+    <xacro:odri_dual_motor_testbed_gazebo  name="picodualdrv8316c"/>
+  </xacro:if>
+  <xacro:unless value="$(arg gz_sim)">
+    <xacro:include filename="$(find odri_dual_motor_testbed_description)/ros2_control/system_pico_dual_drv8316c.ros2_control.xacro" />
+    <xacro:pico_dual_drv8316c_ros2_control
+        name="picodualdrv8316c"
+        />
+  </xacro:unless>
 </robot>

File: odri_dual_motor_testbed_description/robots/fivebar_2dof_robot.urdf.xacro (robot description, xacro)
@@ -9,4 +9,5 @@
        single-robot behaviour is unchanged. -->
   <xacro:arg name="robot_namespace" default=""/>
+  <xacro:arg name="gz_sim" default="false"/>
   <!-- Controller manager parameters file loaded by the odri_gz_ros2_control
        plugin. Defaults to the single-robot forward-command-controller setup
@@ -14,6 +15,4 @@
        controller set (e.g. odri_five_bar_force_velocity_controller for the
        haptic pair). -->
-  <xacro:arg name="controller_params_file"
-             default="$(find odri_dual_motor_testbed_gazebo)/config/forward_command_controller.yaml"/>
   <link name="world"/>
   <xacro:include filename="$(find odri_dual_motor_testbed_description)/urdf/fivebar_2dof.urdf.xacro" />
@@ -23,4 +22,15 @@
     <origin xyz="0.0 0.0 0.001" rpy ="0.0 0.0 0.0"/>
   </joint>
-  <xacro:include filename="$(find odri_dual_motor_testbed_description)/ros2_control/system_pico_dual_drv8316c.ros2_control.xacro" />
+  <xacro:if value="$(arg gz_sim)">
+    <xacro:include filename="$(find odri_dual_motor_testbed_description)/gazebo/gazebo_fivebard_2dof.urdf.xacro" />
+    <xacro:odri_dual_motor_testbed_gazebo
+        name="picodualdrv8316c"
+        />
+  </xacro:if>
+  <xacro:unless value="$(arg gz_sim)">
+    <xacro:include filename="$(find odri_dual_motor_testbed_description)/ros2_control/system_pico_dual_drv8316c.ros2_control.xacro" />
+    <xacro:pico_dual_drv8316c_ros2_control
+        name="picodualdrv8316c"
+        />
+  </xacro:unless>
 </robot>

File: odri_dual_motor_testbed_description/urdf/fivebar_2dof.urdf.xacro (robot description, xacro)
@@ -470,78 +470,3 @@
     <axis xyz="0 0 1"/>
   </joint>
-  <ros2_control name="GazeboOdriSimSystem" type="system">
-    <hardware>
-      <plugin>odri_gz_ros2_control/GazeboOdriSimSystem</plugin>
-    </hardware>
-    <joint name="motor_1">
-      <command_interface name="position" />
-      <command_interface name="velocity" />
-      <command_interface name="effort" />
-      <command_interface name="gain_kp" />
-      <command_interface name="gain_kd" />
-      <state_interface name="velocity" />
-      <state_interface name="position" />
-      <state_interface name="effort" />
-    </joint>
-    <joint name="motor_2">
-      <command_interface name="position" />
-      <command_interface name="velocity" />
-      <command_interface name="effort" />
-      <command_interface name="gain_kp" />
-      <command_interface name="gain_kd" />
-      <state_interface name="velocity" />
-      <state_interface name="position" />
-      <state_interface name="effort" />
-    </joint>
-    <joint name="passive_1">
-      <state_interface name="velocity" />
-      <state_interface name="position" />
-      <state_interface name="effort" />
-    </joint>
-    <joint name="passive_2">
-      <state_interface name="velocity" />
-      <state_interface name="position" />
-      <state_interface name="effort" />
-    </joint>
-  </ros2_control>
-  <gazebo>
-    <plugin filename="odri_gz_ros2_control-system" name="odri_gz_ros2_control::GazeboOdriSimROS2ControlPlugin">
-      <parameters>$(arg controller_params_file)</parameters>
-      <ros>
-        <namespace>$(arg robot_namespace)</namespace>
-      </ros>
-    </plugin>
-  </gazebo>
-  <!-- ================================================================ -->
-  <!--      Gazebo Harmonic (gz-sim8) system plugin for five-bar loop closure. -->
-  <!--      Exact direct geometric model: reads motor_1/motor_2 and imposes -->
-  <!--      passive_1/passive_2 via Joint::ResetPosition every step. -->
-  <!--      See five_bar_mgd_spec.md at the repository root. -->
-  <!--      ================================================================ -->
-  <gazebo>
-    <plugin filename="libFiveBarClosurePlugin.so"
-            name="odri_gz::FiveBarClosurePlugin">
-      <!-- Actuated joints (inputs, theta1/theta2). -->
-      <motor_joint1>motor_1</motor_joint1>
-      <motor_joint2>motor_2</motor_joint2>
-      <!-- Passive joints (outputs, beta1/beta2), imposed exactly. -->
-      <elbow_joint1>passive_1</elbow_joint1>
-      <elbow_joint2>passive_2</elbow_joint2>
-      <!-- Geometry parameters, re-derived from MOTKINBENCH robot.urdf and
-           verified numerically (worst loop-closure residual 6.6e-07 m over
-           theta in [-0.7, 0.7]^2). The plugin's a_x/a_z/b_x/b_z naming is
-           historical: for this robot the plane is (x,y) of `case`, so a_z/b_z
-           carry the y coordinates. See five_bar_mgd_spec.md section 2. -->
-      <a_x>-0.0421006</a_x>
-      <a_z>0.0302628</a_z>
-      <b_x>0.0578994</b_x>
-      <b_z>0.0302628</b_z>
-      <l1>0.06</l1>
-      <l2>0.1</l2>
-      <phi1>2.2329993267948964</phi1>
-      <phi2>1.5045472267948965</phi2>
-      <psi1>0.8742569999992758</psi1>
-      <psi2>2.4450572629561456</psi2>
-    </plugin>
-  </gazebo>
 </robot>
