Commit message: [odri_dual_motor_testbed_description] Fix collision problem with the fivebar model.

File: odri_dual_motor_testbed_description/gazebo/gazebo_fivebar_2dof.urdf.xacro (robot description, xacro)
@@ -104,4 +104,37 @@
     </plugin>
   </gazebo>
+  <!-- ================================================================ -->
+  <!--      Collision filtering. Contacts only occur between two collisions -->
+  <!--      whose collide_bitmask values share a bit. These must be set here, -->
+  <!--      through <gazebo reference>: a <surface> tag inside a URDF -->
+  <!--      <collision> is dropped by the URDF to SDF conversion. -->
+  <!--      The base is welded to the world: without mask 0 its meshes touch -->
+  <!--      the ground plane and the contact computation slows the simulation -->
+  <!--      down about 50 times. -->
+  <!--      ================================================================ -->
+  <!-- Base, welded to the world: no contact. -->
+  <gazebo reference="case">
+    <collision><surface><contact><collide_bitmask>0x00</collide_bitmask></contact></surface></collision>
+  </gazebo>
+  <!-- Base, welded to the world: no contact. -->
+  <gazebo reference="top_cover">
+    <collision><surface><contact><collide_bitmask>0x00</collide_bitmask></contact></surface></collision>
+  </gazebo>
+  <!-- Left crank. -->
+  <gazebo reference="rotor">
+    <collision><surface><contact><collide_bitmask>0x04</collide_bitmask></contact></surface></collision>
+  </gazebo>
+  <!-- Left coupler. -->
+  <gazebo reference="arm_l2">
+    <collision><surface><contact><collide_bitmask>0x01</collide_bitmask></contact></surface></collision>
+  </gazebo>
+  <!-- Right crank. -->
+  <gazebo reference="rotor_2">
+    <collision><surface><contact><collide_bitmask>0x08</collide_bitmask></contact></surface></collision>
+  </gazebo>
+  <!-- Right coupler: no bit in common with the other moving links, so the arms never collide with each other. -->
+  <gazebo reference="arm_r2">
+    <collision><surface><contact><collide_bitmask>0x02</collide_bitmask></contact></surface></collision>
+  </gazebo>
   </xacro:macro>
 </robot>

File: odri_dual_motor_testbed_description/urdf/fivebar_2dof.urdf.xacro (robot description, xacro)
@@ -20,6 +20,8 @@
   3. The stray empty link c_0402_1005metric (a KiCad footprint that leaked
      into the CAD assembly; 1e-9 mass, no visual, no collision) is dropped.
-  4. collide_bitmask surface tags added on the four moving links, carried over
-     from the previous revision of this file, so the arms never self-collide.
+  4. Collision filtering (collide_bitmask) is set in
+     gazebo/gazebo_fivebar_2dof.urdf.xacro, through <gazebo reference> blocks:
+     a <surface> tag inside a URDF <collision> is dropped by the URDF to SDF
+     conversion.
   5. ros2_control + Gazebo plugin blocks appended (not part of the export).
   6. motor_1 / motor_2 origin yaw set to 0 (exported: 0.662203 / -0.0662491),
@@ -210,9 +212,4 @@
         <mesh filename="package://odri_dual_motor_testbed_description/meshes/assets/five_bar/rotor.stl"/>
       </geometry>
-      <surface>
-        <contact>
-          <collide_bitmask>0x04</collide_bitmask>
-        </contact>
-      </surface>
     </collision>
     <!-- Part arm_l1 -->
@@ -231,9 +228,4 @@
         <mesh filename="package://odri_dual_motor_testbed_description/meshes/assets/five_bar/arm_l1.stl"/>
       </geometry>
-      <surface>
-        <contact>
-          <collide_bitmask>0x04</collide_bitmask>
-        </contact>
-      </surface>
     </collision>
   </link>
@@ -260,9 +252,4 @@
         <mesh filename="package://odri_dual_motor_testbed_description/meshes/assets/five_bar/arm_l2.stl"/>
       </geometry>
-      <surface>
-        <contact>
-          <collide_bitmask>0x01</collide_bitmask>
-        </contact>
-      </surface>
     </collision>
   </link>
@@ -334,9 +321,4 @@
         <mesh filename="package://odri_dual_motor_testbed_description/meshes/assets/five_bar/arm_r1.stl"/>
       </geometry>
-      <surface>
-        <contact>
-          <collide_bitmask>0x08</collide_bitmask>
-        </contact>
-      </surface>
     </collision>
     <!-- Part rotor_2 -->
@@ -355,9 +337,4 @@
         <mesh filename="package://odri_dual_motor_testbed_description/meshes/assets/five_bar/rotor.stl"/>
       </geometry>
-      <surface>
-        <contact>
-          <collide_bitmask>0x08</collide_bitmask>
-        </contact>
-      </surface>
     </collision>
   </link>
@@ -384,9 +361,4 @@
         <mesh filename="package://odri_dual_motor_testbed_description/meshes/assets/five_bar/arm_r2.stl"/>
       </geometry>
-      <surface>
-        <contact>
-          <collide_bitmask>0x02</collide_bitmask>
-        </contact>
-      </surface>
     </collision>
   </link>
