Commit message: pico -> motkin

File: motkin_dual_motor_testbed_description/robots/dual_flywheel_robot.urdf.xacro (robot description, xacro)
@@ -9,5 +9,5 @@
        single-robot behaviour is unchanged. -->
   <xacro:arg name="robot_namespace" default=""/>
-  <!-- Serial device of the pico_dual_drv8316c board on the real robot.
+  <!-- Serial device of the motkin board on the real robot.
        Empty: auto-detected. Set it when several testbeds are connected to
        the same computer, e.g. /dev/serial/by-id/usb-...  -->
@@ -29,7 +29,7 @@
   </xacro:if>
   <xacro:unless value="$(arg gz_sim)">
-    <xacro:include filename="$(find motkin_dual_motor_testbed_description)/ros2_control/system_pico_dual_drv8316c.ros2_control.xacro" />
-    <xacro:pico_dual_drv8316c_ros2_control
-        name="picodualdrv8316c"
+    <xacro:include filename="$(find motkin_dual_motor_testbed_description)/ros2_control/system_motkin.ros2_control.xacro" />
+    <xacro:motkin_ros2_control
+        name="motkin"
         serial_port="$(arg serial_port)"
         />

File: motkin_dual_motor_testbed_description/robots/fivebar_2dof_robot.urdf.xacro (robot description, xacro)
@@ -9,5 +9,5 @@
        single-robot behaviour is unchanged. -->
   <xacro:arg name="robot_namespace" default=""/>
-  <!-- Serial device of the pico_dual_drv8316c board on the real robot.
+  <!-- Serial device of the motkin board on the real robot.
        Empty: auto-detected. Set it when several testbeds are connected to
        the same computer, e.g. /dev/serial/by-id/usb-...  -->
@@ -32,7 +32,7 @@
   </xacro:if>
   <xacro:unless value="$(arg gz_sim)">
-    <xacro:include filename="$(find motkin_dual_motor_testbed_description)/ros2_control/system_pico_dual_drv8316c.ros2_control.xacro" />
-    <xacro:pico_dual_drv8316c_ros2_control
-        name="picodualdrv8316c"
+    <xacro:include filename="$(find motkin_dual_motor_testbed_description)/ros2_control/system_motkin.ros2_control.xacro" />
+    <xacro:motkin_ros2_control
+        name="motkin"
         five_bar="true"
         serial_port="$(arg serial_port)"

File: motkin_dual_motor_testbed_description/ros2_control/system_motkin.ros2_control.xacro (robot description, xacro)
@@ -6,6 +6,5 @@
     system_dual_motor_testbed.ros2_control.xacro: same joint names and same
     position/velocity/effort/gain_kp/gain_kd interfaces, but backed by a
-    pico_dual_PMSM_BUG79100G_DRV8316C board over USB instead of an MOTKIN
-    master board over Ethernet or Gazebo.
+    motkin board over USB instead of  Gazebo.
     serial_port: left empty to auto-detect (/dev/serial/by-id, then
     /dev/ttyACM*, then /dev/ttyUSB*), or set explicitly, e.g. /dev/ttyACM0.
@@ -17,5 +16,5 @@
     gazebo/gazebo_fivebar_2dof.urdf.xacro (see five_bar_mgd_spec.md).
   -->
-  <xacro:macro name="pico_dual_drv8316c_ros2_control"
+  <xacro:macro name="motkin_ros2_control"
                params="name
                        left_joint_name:=motor_1
@@ -29,5 +28,5 @@
         <xacro:if value="${five_bar}">
           <plugin>motkin_dual_motor_testbed_hardware/FiveBarSystem</plugin>
-          <param name="inner_plugin">pico_dual_drv8316c_hardware_interface/SystemPicoDualDrv8316CHardware</param>
+          <param name="inner_plugin">motkin_ros2_hardware_interface/SystemPicoDualDrv8316CHardware</param>
           <param name="motor_joint1">${left_joint_name}</param>
           <param name="motor_joint2">${right_joint_name}</param>
@@ -46,5 +45,5 @@
         </xacro:if>
         <xacro:unless value="${five_bar}">
-          <plugin>pico_dual_drv8316c_hardware_interface/SystemPicoDualDrv8316CHardware</plugin>
+          <plugin>motkin_ros2_hardware_interface/SystemPicoDualDrv8316CHardware</plugin>
         </xacro:unless>
         <param name="serial_port">${serial_port}</param>

File: motkin_dual_motor_testbed_description/urdf/dual_flywheel.urdf.xacro (robot description, xacro)
@@ -13,5 +13,5 @@
      same as for the five-bar model (see fivebar_2dof.urdf.xacro).
   3. The ros2_control block + motkin_gz_ros2_control plugin live in
-     ros2_control/system_pico_dual_drv8316c.ros2_control.xacro, included
+     ros2_control/system_motkin.ros2_control.xacro, included
      separately by robots/dual_flywheel_robot.urdf.xacro.
   This mechanism has no closed kinematic loop: motor_1/motor_2 directly
